File: PCB/Kicad/THT_SolderTypeDB19/BurgerDisk_THT_SolderTypeDB19.kicad_pcb (KiCad board)
At the start: 2 copper layers, 93.7 x 67.6 mm, 17 parts, among them J1 Daisy port in, J2 MicroSD module, J3 UART, J4 Daisy port out, U1 PC817

Commit message: Modify holder a bit
Parts:
- added REF**: MountingHole_8.4mm_M8, MountingHole:MountingHole_8.4mm_M8, F.Cu at (157.0, 101.3)
Changed lines of the file:
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@@
+  )
+  (footprint "MountingHole:MountingHole_8.4mm_M8" (layer "F.Cu")
+    (at 156.972 101.346)
+    (descr "Mounting Hole 8.4mm, no annular, M8")
+    (tags "mounting hole 8.4mm no annular m8")
+    (attr board_only exclude_from_pos_files exclude_from_bom)
+    (fp_text reference "REF**" (at 0 -9.4) (layer "F.Fab")
+        (effects (font (size 1 1) (thickness 0.15)))
+    )
+    (fp_text value "MountingHole_8.4mm_M8" (at 0 9.4) (layer "F.Fab")
+        (effects (font (size 1 1) (thickness 0.15)))
+    )
+    (fp_text user "${REFERENCE}" (at 0 0) (layer "F.Fab")
+        (effects (font (size 1 1) (thickness 0.15)))
+    )
+    (fp_circle (center 0 0) (end 8.4 0)
+      (stroke (width 0.15) (type solid)) (fill none) (layer "Cmts.User"))
+    (fp_circle (center 0 0) (end 8.65 0)
+      (stroke (width 0.05) (type solid)) (fill none) (layer "F.CrtYd"))
+    (pad "" np_thru_hole circle (at 0 0) (size 8.4 8.4) (drill 8.4) (layers "*.Cu" "*.Mask"))
   )
   (footprint "MountingHole:MountingHole_8.4mm_M8" (layer "F.Cu")

Commit message: Small esthetic fixes
Other:
- board text added: "+5V/GND"
Changed lines of the file:
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@@
         (effects (font (size 1 1) (thickness 0.15)))
     )
-    (fp_text value "MicroSD module" (at 4.385 14.97 -90) (layer "F.SilkS")
+    (fp_text value "MicroSD module" (at -2.794 10.922) (layer "F.SilkS")
         (effects (font (size 1 1) (thickness 0.15)))
     )
@@
   (gr_rect (start 70.866 43.688) (end 164.592 111.252)
     (stroke (width 0.05) (type default)) (fill none) (layer "Edge.Cuts"))
+  (gr_text "+5V/GND" (at 141.478 97.282) (layer "F.SilkS")
+    (effects (font (size 1 1) (thickness 0.2) bold) (justify left bottom))
+  )
   (gr_text "BurgerDisk\nDaisy-chainable Apple II Smartport hard drive\n© Colin Leroy-Mira, 2026 - CC BY-SA\nhttps://github.com/colinleroy/BurgerDisk" (at 73.152 56.896) (layer "F.SilkS")
     (effects (font (size 1.5 1.5) (thickness 0.3) bold) (justify left bottom))
