File: PCB/Smallest/Smallest.kicad_sch (KiCad schematic)
At the start: 30 parts, among them J1 Daisy port in, J2 ICSP_ISP6, J3 UART, J4 Daisy port out, K1 HYC77-TF09-200, U1 PC817C-S, U2 SE5218, U21 TXB0104QPWRQ1, U3 ATmega328P-AU, Y1 16MHz

Commit message: WIP untested very small PCB
Parts:
- removed J1: Daisy port in, Connector_IDC:IDC-Header_2x10_P2.54mm_Vertical, symbol Connector_Generic:Conn_02x10_Odd_Even
- added J4: Daisy port in, db19:DSUB-19_Male_EdgeMount_Pitch2.77mm, symbol db19:DB19_Male
- D3: renamed from D4; footprint LED_THT:LED_D3.0mm -> LED_SMD:LED_0603_1608Metric; LCSC C5875763 -> C2288
- J1: renamed from J4; footprint DSUB-19-angled:DSUB-19_Female_Horizontal_MXS82009-8251-9246 -> db19:DSUB-19_Female_EdgeMount_Pitch2.77mm
- J2: footprint Connector_IDC:IDC-Header_2x03_P2.54mm_Vertical -> Connector_IDC:IDC-Header_2x03_P2.54mm_Vertical_SMD; LCSC C11214 -> C192301
- renumbered C9 to C1, C6 to C10, C8 to C2, C10 to C3, C5 to C4, C1 to C5, C2 to C6, C3 to C7, C4 to C8, C7 to C9, D3 to D1, R3 to R1, R4 to R2, R5 to R3, R7 to R4, R1 to R5, R2 to R6, R6 to R7, U3 to U2, U2 to U3, U21 to U4
Connections:
- net +12V: now also J4.7, J4.8
- net -12V: now also J4.5
- net 5V_apple2: now also J4.6
- net DRV1_in: now also J4.17 (P17)
- net DRV2_in: now also J4.9
- net EN3.5: now also J4.4
- net GND: now also J4.1, J4.2, J4.3; no longer J1.0
- net HDSEL_in: now also J4.16 (P16)
- net PH0: now also J4.11 (P11)
- net PH1: now also J4.12 (P12)
- net PH2: now also J4.13 (P13)
- net PH3_in: now also J4.14 (P14)
- net WRDATA: now also J4.19 (P19)
- net WREQ: now also J4.15 (P15)
- net WRPROT_out: now also J4.10
- net RDDATA_in renamed RDDATA
- net RDDATA: now also J4.18 (P18)
- no-connect marks 8 -> 7
Other:
- note added: "APPLE II INTERFACE"
- note added: "MICROSD LEVEL SHIFTER"
- note added: "MICROSD VOLTAGE REGULATOR"
- note added: "MINIMAL ATMEGA328"
- note removed: "HEADER"
- note removed: "VOLTAGE LEVEL TRANSLATOR"
- note removed: "VOLTAGE REGULATOR"
- title: BurgerDisk PCB - Angled DB19 version -> DominoDisk - very small Apple II hard drive
- moved on the sheet: C1, C10, C2, C3, C4, C5, C6, C7, C8, C9, D1, D2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
