File: PCB/BurgerDisk-THT-SolderTypeDB19/BurgerDisk-THT-SolderTypeDB19.kicad_sch (KiCad schematic)
At the start: 14 parts, among them J1 Daisy port in, J2 MicroSD module, J3 UART, J4 Daisy port out, U1 PC817

Commit message: Add logo (thanks to Javier Rivera!!)
Add my own micro/SD modules
Parts:
- J2: LCSC C6209271 -> C56816
Changed lines of the file:
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@@
 			)
 		)
-		(property "LCSC" "C6209271"
+		(property "LCSC" "C56816"
 			(at 99.06 132.08 0)
 			(effects

Commit message: Add indicator on PC817 pin1
Parts:
- D4, J3: LCSC C6273326 -> C32713268
Changed lines of the file:
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@@
 			)
 		)
-		(property "LCSC" "C6273326"
+		(property "LCSC" "C32713268"
 			(at 222.25 27.94 0)
 			(effects
@@
 			)
 		)
-		(property "LCSC" "C6273326"
+		(property "LCSC" "C32713268"
 			(at 195.58 113.03 0)
 			(effects
