File: PCB/BurgerDisk-THT-AngledDB19/BurgerDisk-THT-AngledDB19.kicad_pcb (KiCad board)
At the start: 2 copper layers, 93.7 x 73.4 mm, 18 parts, among them J1 Daisy port in, J2 MicroSD module, J3 UART, J4 Daisy port out, U1 PC817

Commit message: Update details
Routing:
- net GND: track 56.7 -> 10.6 mm
- net DRV2_in: track 44.8 -> 45.8 mm
- net DRV2_out: track 122.7 -> 121.8 mm
- net Net-(R3-Pad2): track 20.5 -> 19.7 mm
- net +12V: track 53.7 -> 53.0 mm
- net TX: track 12.1 -> 11.4 mm
- net HDSEL_in: track 9.78 -> 9.16 mm
- net Net-(R4-Pad2): track 18.3 -> 18.9 mm
