File: PCB/Small-atmega-SMD/Small-atmega-SMD.kicad_pcb (KiCad board)
At the start: 2 copper layers, 65.1 x 96.9 mm, 35 parts, among them J1 Daisy port out, J2 ICSP_ISP6, J3 2-pin header, J4 Daisy port in, J5 Ext. MicroSD module, J6 2-pin header, K1 HYC77-TF09-200, U1 PC817C-S, U2 ATmega328P-AU, U3 SE5218, U4 TXB0104PWR, Y1 Resonator_GND2

Commit message: OCD
Parts:
- moved D2 19.8 mm to (122.0, 66.9), turned to 180 degrees
- moved C5 11.2 mm to (114.6, 113.8), turned to 0 degrees
- moved JP1 9.29 mm to (112.4, 79.3), turned to -90 degrees
- moved C4 9.08 mm to (110.1, 113.8), turned to 0 degrees
- moved J3 8.90 mm to (105.3, 71.9)
- moved JP2 7.26 mm to (112.3, 83.5)
- moved C2 5.56 mm to (109.6, 101.2), turned to 180 degrees
- moved U4 5.23 mm to (112.5, 110.2), turned to 180 degrees
- moved C3 4.21 mm to (112.6, 101.2), turned to 0 degrees
- moved U1 2.12 mm to (137.3, 65.1)
- moved D1 1.99 mm to (136.9, 58.1)
- moved R2 1.89 mm to (142.6, 60.9)
- moved R1 1.76 mm to (141.0, 60.9)
- moved R4 1.68 mm to (136.7, 73.2)
- moved R3 1.40 mm to (122.1, 68.6)
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- renumbered C3 to C2, C2 to C3, D4 to D3, JP2 to JP1, JP1 to JP2
Routing:
- net WRPROT_out: track 68.0 -> 112.8 mm, vias 1 -> 0
- net GND: track 61.8 -> 34.3 mm, vias 8 -> 5
- net LED: track 98.1 -> 82.2 mm
- net WRPROT_in: track 17.5 -> 2.36 mm, vias 2 -> 0
- net 3V3: track 51.4 -> 40.0 mm
- net 5V_intMicroSD: track 27.2 -> 36.8 mm, vias 2 -> 0
- net CS_L: track 34.7 -> 25.9 mm
- net RDDATA: track 76.2 -> 67.6 mm
- net Net-(JP2-A): track 55.7 -> 64.3 mm, vias 0 -> 2
- net TX: track 10.1 -> 18.5 mm
- net MOSI_L: track 33.1 -> 25.5 mm
- net EN3.5: track 66.0 -> 58.7 mm
- net WREQ: track 66.3 -> 59.3 mm
- net WRDATA: track 77.7 -> 70.9 mm
- net SCLK_L: track 30.8 -> 24.5 mm
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Other:
- board text added: "CUT FOR EXTERNAL LED+RESISTOR"
- board text added: "If using an external SD or MicroSD module, cut power to the internal one by cutting the trace in the JP2 jumper. If using an external LED (with external resistor), cut power to the internal one by cutting the trace in the JP1 jumper."
- board text removed: "CUT FOR EXT LED"
- board text removed: "If using an external SD or MicroSD module, cut power to the internal one by cutting the trace in the JP1 jumper. If using an external LED (with external resistor), cut power to the internal one by cutting the trace in the JP2 jumper."
