File: PCB/Small-atmega-SMD/Small-atmega-SMD.kicad_sch (KiCad schematic)
At the start: 30 parts, among them J1 Daisy port out, J2 ICSP_ISP6, J3 2-pin header, J4 Daisy port in, J5 Ext. MicroSD module, J6 2-pin header, K1 HYC77-TF09-200, U1 PC817C-S, U2 ATmega328P-AU, U3 SE5218, U4 TXB0104PWR, Y1 Resonator_GND2

Commit message: OCD
Parts:
- J5: LCSC (none) -> C56816
- renumbered C3 to C2, C2 to C3, D4 to D3, JP2 to JP1, JP1 to JP2
Changed lines of the file:
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@@
 		(on_board yes)
 		(dnp no)
-		(property "Reference" "C2"
+		(property "Reference" "C3"
 			(at 260.35 147.32 90)
 			(effects
@@
 			(project "Small"
 				(path "/596d0583-1d97-453e-b84c-75eed809afa2"
-					(reference "C2")
+					(reference "C3")
 					(unit 1)
 				)
@@
 		(dnp no)
 		(fields_autoplaced yes)
-		(property "Reference" "JP1"
+		(property "Reference" "JP2"
 			(at 236.22 124.4599 90)
 			(effects
@@
 			(project ""
 				(path "/596d0583-1d97-453e-b84c-75eed809afa2"
-					(reference "JP1")
+					(reference "JP2")
 					(unit 1)
 				)
@@
 					(size 1.27 1.27)
 				)
+			)
+		)
+		(property "LCSC" "C56816"
+			(at 189.23 41.91 0)
+			(effects
+				(font
+					(size 1.27 1.27)
+				)
+				(hide yes)
 			)
 		)
@@
 		(dnp no)
 		(fields_autoplaced yes)
-		(property "Reference" "JP2"
+		(property "Reference" "JP1"
 			(at 152.4 125.7299 90)
 			(effects
@@
 			(project "Small-atmega-SMD"
 				(path "/596d0583-1d97-453e-b84c-75eed809afa2"
-					(reference "JP2")
+					(reference "JP1")
 					(unit 1)
 				)
@@
 		(on_board yes)
 		(dnp no)
-		(property "Reference" "C3"
+		(property "Reference" "C2"
 			(at 229.87 148.59 90)
 			(effects
@@
 			(project "Small"
 				(path "/596d0583-1d97-453e-b84c-75eed809afa2"
-					(reference "C3")
+					(reference "C2")
 					(unit 1)
 				)
@@
 		(dnp no)
 		(fields_autoplaced yes)
-		(property "Reference" "D4"
+		(property "Reference" "D3"
 			(at 153.67 142.5574 90)
 			(effects
@@
 			)
 		)
-		(property "Description" ""
+		(property "Description" "Blue LED, 3mm, 3.3V 20mA"
 			(at 149.86 142.24 0)
 			(effects
@@
 			(project "Small-atmega-SMD"
 				(path "/596d0583-1d97-453e-b84c-75eed809afa2"
-					(reference "D4")
+					(reference "D3")
 					(unit 1)
 				)
@@
 			)
 		)
-		(property "Description" "Three pin crystal, GND on pin 2"
+		(property "Description" "CSTNE16M0V530000R0"
 			(at 102.87 135.89 0)
 			(effects

Commit message: Fix details on DD/angled
Parts:
- J5: LCSC C56816 -> (none)
- J6: LCSC C32713268 -> (none)
Changed lines of the file:
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@@
-			)
-		)
-		(property "LCSC" "C56816"
-			(at 189.23 41.91 0)
-			(effects
-				(font
-					(size 1.27 1.27)
-				)
-				(hide yes)
 			)
 		)
@@
 			)
 		)
-		(property "LCSC" "C32713268"
+		(property "LCSC" ""
 			(at 165.1 140.97 0)
 			(effects
