File: PCB/BurgerDisk-SMD/BurgerDisk-SMD.kicad_sch (KiCad schematic)
At the start: 18 parts, among them J1 Daisy port out, J2 2-pin header, J3 ICSP_ISP6, J4 Daisy port in, J5 MicroSD module, U1 PC817C-S, U2 ATmega328P-AU, Y1 Resonator_GND2

Commit message: Move to bigger pads for diodes
Parts:
- D1: footprint Diode_SMD:D_SOD-323F -> Diode_SMD:D_SOD-323_HandSoldering
- D2: footprint Diode_SMD:D_SOD-323 -> Diode_SMD:D_SOD-323_HandSoldering
Changed lines of the file:
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@@
 			)
 		)
-		(property "Footprint" "Diode_SMD:D_SOD-323F"
+		(property "Footprint" "Diode_SMD:D_SOD-323_HandSoldering"
 			(at 67.31 61.595 0)
 			(effects
@@
 			)
 		)
-		(property "Footprint" "Diode_SMD:D_SOD-323"
+		(property "Footprint" "Diode_SMD:D_SOD-323_HandSoldering"
 			(at 146.05 109.855 0)
 			(effects
