File: PCB/BurgerDisk-SMD/BurgerDisk-SMD.kicad_pcb (KiCad board)
At the start: 2 copper layers, 65.1 x 96.9 mm, 23 parts, among them J1 Daisy port out, J2 2-pin header, J3 ICSP_ISP6, J4 Daisy port in, J5 MicroSD module, U1 PC817C-S, U2 ATmega328P-AU, Y1 Resonator_GND2

Commit message: Align
Parts:
- moved R4 2.50 mm to (141.5, 73.0)
- moved R3 0.76 mm to (141.5, 74.5)
Routing:
- net DRV2_in: track 44.5 -> 42.8 mm
- net DRV2_burgerDisk: track 13.4 -> 12.2 mm
- net Net-(R3-Pad2): track 6.45 -> 5.20 mm
- net 5V_burgerDisk: track 134.9 -> 134.2 mm
