File: PCB/Mini-SMD-Angled/Mini-SMD-Angled.kicad_sch (KiCad schematic)
At the start: 30 parts, among them J1 Daisy port out, J2 ICSP_ISP6, J3 2-pin header, J4 Daisy port in, J5 Ext. MicroSD module, J6 2-pin header, K1 HYC77-TF09-200, U1 PC817C-S, U2 ATmega328P-AU, U3 SE5218, U4 TXB0104PWR, Y1 Resonator_GND2

Commit message: Move to bigger pads for diodes
Parts:
- D1: footprint Diode_SMD:D_SOD-323 -> Diode_SMD:D_SOD-323_HandSoldering
- D2: footprint Diode_SMD:D_SOD-323F -> Diode_SMD:D_SOD-323_HandSoldering
Changed lines of the file:
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@@
 			)
 		)
-		(property "Footprint" "Diode_SMD:D_SOD-323F"
+		(property "Footprint" "Diode_SMD:D_SOD-323_HandSoldering"
 			(at 67.31 61.595 0)
 			(effects
@@
 			)
 		)
-		(property "Footprint" "Diode_SMD:D_SOD-323"
+		(property "Footprint" "Diode_SMD:D_SOD-323_HandSoldering"
 			(at 146.05 109.855 0)
 			(effects
