File: PCB/DB19-IDC20-Adapter/DB19-IDC20-Adapter.kicad_pcb (KiCad board)
At the start: 2 copper layers, 4 parts, among them J1 DB19, J2 IDC20

Commit message: Cleanups
Routing:
- net GND: track 30.0 -> 0.00 mm
- net +12V: track 19.3 -> 24.6 mm
Other:
- board outline added: 41 x 18.1 mm

Commit message: Cleanups
Other:
- board text added: "BurgerDisk IDC20/DB19 adapter For Apple II only"
- board text added: "DB19M"
