File: PCB/MicroSD-module/MicroSD-module.kicad_pcb (KiCad board)
At the start: 2 copper layers, 24.4 x 41.9 mm, 14 parts, among them J1 Connector, K1 HYC77-TF09-200, U1 SE5218, U2 TXB0104PWR

Commit message: Cleanups
Routing:
- net GND: track 28.4 -> 11.3 mm
- net MOSI: track 13.4 -> 12.4 mm
- net MISO: track 12.3 -> 13.0 mm
