File: PCB/BurgerDisk-SMD-Angled/BurgerDisk-SMD-Angled.kicad_pcb (KiCad board)
At the start: 2 copper layers, 65.1 x 96.9 mm, 23 parts, among them J1 Daisy port out, J2 2-pin header, J3 ICSP_ISP6, J4 Daisy port in, J5 MicroSD module, U1 PC817C-S, U2 ATmega328P-AU, Y1 Resonator_GND2

Commit message: Cleanups
Parts:
- J1: footprint db19:DSUB-19_Female_EdgeMount_Pitch2.77mm -> DSUB-19-angled:DSUB-19_Female_Horizontal_MXS82009-8251-9246
- moved J1 13.1 mm to (128.5, 54.0)
Routing:
- net +12V: track 67.5 -> 64.5 mm
- net DRV2_out: track 29.1 -> 26.8 mm, vias 2 -> 1
- net 5V_apple2: track 64.9 -> 62.7 mm
- net WRPROT_out: track 79.6 -> 77.4 mm
- net -12V: track 66.4 -> 64.8 mm
- net EN3.5: track 69.3 -> 67.8 mm
- net RDDATA: track 80.9 -> 79.9 mm
- net WRDATA: track 80.6 -> 81.3 mm
Other:
- outline, holes or cut-outs redrawn

Commit message: Align
Parts:
- moved R4 2.32 mm to (141.5, 73.2)
- moved R3 0.84 mm to (141.5, 74.7)
Routing:
- net DRV2_burgerDisk: track 13.4 -> 12.3 mm
- net Net-(R3-Pad2): track 6.45 -> 7.30 mm
